File: Emaplaat_ja_ekraan/emaplaat_ja_ekraan.kicad_pcb (KiCad board)
At the start: 2 copper layers, 1 part, among them U1 ESP32-S3-WROOM-2

Commit message: Urmas Tamm
Parts:
- removed U1: ESP32-S3-WROOM-2, RF_Module:ESP32-S3-WROOM-2
- added IC1: TPS54429PWPR, SOP65P640X120-15N:SOP65P640X120-15N, F.Cu at (102.2, 130.2)
- added IC2: ESP32-S3-WROOM-2-N32R16V, ESP32S3WROOM2N32R16V:ESP32S3WROOM2N32R16V, F.Cu at (93.3, 96.5)
- added IC3: FT232RNL-TUBE, SOP65P780X200-28N:SOP65P780X200-28N, F.Cu at (125.0, 129.3)
- added J2: USB4216-03-A, USB421603A:USB421603A, F.Cu at (127.3, 118.4)
- added S1: TL3305BF100QG, TL3305BF160QG:TL3305BF160QG, F.Cu at (125.8, 101.5)
- added S2: TL3305BF100QG, TL3305BF160QG:TL3305BF160QG, F.Cu at (125.8, 109.2)
