File: Ekraan_7x7/array.kicad_sch (KiCad schematic)
At the start: 36 parts, among them IC12 1EDN7550BXTSA1, IC13 1EDN7550BXTSA1, IC14 1EDN7550BXTSA1, IC15 1EDN7550BXTSA1, IC2 1EDN7550BXTSA1, IC4 1EDN7550BXTSA1, IC5 1EDN7550BXTSA1, U2 1EDN7550BXTSA1

Commit message: Koomas Plank
Parts:
- removed C11, C14, C20, C23, C25: 22u, symbol Device:C
- removed IC12, IC13, IC14: 1EDN7550BXTSA1, SOT95P280X145-6N, symbol 1EDN7550BXTSA1:1EDN7550BXTSA1
- removed R21, R22, R23, R24, R25, R26: 33k, symbol Device:R
- added C2, C48, C5, C64, C81: 100u, symbol Device:C
- added IC26, IC28, IC41: 1EDN7550BXTSA1, SOT95P280X145-6N, symbol 1EDN7550BXTSA1:1EDN7550BXTSA1
- added R49, R50, R53, R54, R79, R80: 33k, symbol Device:R
- C10, C27: value 22u -> 100u
- C12: footprint Capacitor_SMD:C_0201_0603Metric -> Capacitor_SMD:C_0805_2012Metric_Pad1.18x1.45mm_HandSolder
Connections:
- net 12V: now also IC15.4 (VDD), IC2.4 (VDD), IC4.4 (VDD), IC5.4 (VDD), C2.1, C48.1, C5.1, C64.1, C81.1, IC26.4 (VDD), IC28.4 (VDD), IC41.4 (VDD)
- net 1C+: now also R28.2
- net 1C-: now also R27.2
- net 1D+: now also R54.2
- net 1D-: now also R53.2
- net 1E+: now also R80.2; no longer R28.2
- net 1E-: now also R79.2; no longer R27.2
- net 1G+: now also R50.2
- net 1G-: now also R49.2
- net PGND: now also C10.2, C27.2, C2.2, C48.2, C5.2, C64.2, C81.2, IC26.2 (GND), IC28.2 (GND), IC41.2 (GND)
- net at C22.1: now also IC26.5 (OUT_SRC), IC26.6 (OUT_SNK)
- net at C26.1: now also IC28.5 (OUT_SRC), IC28.6 (OUT_SNK)
- net at IC15.5 (OUT_SRC), IC15.6 (OUT_SNK): now also C24.1; no longer C28.1
- new net: IC28.1 (IN-), R53.1
- new net: IC28.3 (IN+), R54.1
- new net: IC26.1 (IN-), R49.1
- new net: IC26.3 (IN+), R50.1
- new net: IC41.1 (IN-), R79.1
- new net: IC41.3 (IN+), R80.1
- new net: C28.1, IC41.5 (OUT_SRC), IC41.6 (OUT_SNK)
Other:
- note added: "1x7 Flipdot-id kogum"
- note added: "Flipdot-ide juhtimissüsteem"
- moved on the sheet: C10, C12, C13, C21, C22, C24, C26, C28, IC2, R1, R2, U2
