File: Emaplaat/Emaplaat.kicad_sch (KiCad schematic)
At the start: 14 parts, among them IC2 ESP32-S3-WROOM-2-N32R16V, Q1 2N7002K

Commit message: cleanoupp T__W
Other:
- note added: "Buzzer"
- note added: "Ühendused ja toide"
- moved on the sheet: C10, C11, C12, IC2, R2

Commit message: qqwertrewasdfgfdsdfgfdsdfgfdsasdfghgfdsdfghgfdsasdfghgfdsasdfgfew3
Other:
- removed sheet ekraan
Changed lines of the file:
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@@
-	)
-	(sheet
-		(at 249.555 66.675)
-		(size 16.51 38.1)
-		(exclude_from_sim no)
-		(in_bom yes)
-		(on_board yes)
-		(dnp no)
-		(fields_autoplaced yes)
-		(stroke
-			(width 0.1524)
-			(type solid)
-		)
-		(fill
-			(color 0 0 0 0.0000)
-		)
-		(property "Sheetname" "ekraan"
-			(at 249.555 65.9634 0)
-			(effects
-				(font
-					(size 1.27 1.27)
-				)
-				(justify left bottom)
-			)
-		)
-		(property "Sheetfile" "ekraan.kicad_sch"
-			(at 249.555 105.3596 0)
-			(effects
-				(font
-					(size 1.27 1.27)
-				)
-				(justify left top)
-			)
-		)
-		(instances
-			(project "emaplaat_ja_ekraan"
-				(path "/489224c0-ace1-4530-aa61-a5d03adf1434"
-					(page "2")
-				)
-			)
-		)
 	)
 	(sheet
@@
 		)
 		(instances
-			(project "emaplaat_ja_ekraan"
+			(project "Emaplaat"
 				(path "/489224c0-ace1-4530-aa61-a5d03adf1434"
 					(page "3")

Commit message: Getamine addiction
Parts:
- added J2, J7: Screw_Terminal_01x02, symbol Connector:Screw_Terminal_01x02
- added J3, J4: Conn_01x09_Pin, symbol Connector:Conn_01x09_Pin
Connections:
- net 12V: now also J2.2 (Pin_2), J7.2 (Pin_2)
- net 3V3: now also J3.1 (Pin_1), J4.1 (Pin_1)
- net AGND: now also J3.9 (Pin_9), J4.9 (Pin_9)
- net PGND: now also J2.1 (Pin_1), J7.1 (Pin_1)
- net flipdot2-: now reaches IC2.20 (IO12)
- net flipdot2-: now also J4.8 (Pin_8)
- net flipdot2+: now reaches IC2.21 (IO13)
- net flipdot2+: now also J4.7 (Pin_7)
- net !MR1: now reaches IC2.22 (IO14)
- net !MR1: now also IC2.34 (IO41), J3.6 (Pin_6), J4.6 (Pin_6)
- net SHCP1: now reaches IC2.23 (IO21)
- net SHCP1: now also IC2.33 (IO40), J3.5 (Pin_5), J4.5 (Pin_5)
- net STCP1: now reaches IC2.24 (IO47)
- net STCP1: now also IC2.32 (IO39), J3.4 (Pin_4), J4.4 (Pin_4)
- net !OE1: now reaches IC2.25 (IO48)
- net !OE1: now also IC2.31 (IO38), J3.3 (Pin_3), J4.3 (Pin_3)
- net DS1: now reaches IC2.27 (IO0)
- net DS1: now also IC2.39 (IO1), J3.2 (Pin_2), J4.2 (Pin_2)
- net flipdot1+: now reaches IC2.35 (IO42)
- net flipdot1+: now also J3.7 (Pin_7)
- net flipdot1-: now reaches IC2.38 (IO2)
- net flipdot1-: now also J3.8 (Pin_8)
Other:
- note added: "Peamine protsessor, kõik komponendid võetud andmelehest"
- note added: "Sisend ühendused ja toide"
- note added: "kaks 12V ja GND toite kruvi ühendust 7x7 ekraanidele"
- note added: "kaks kontroll ühendust 7x7 ekraanidele"
- note removed: "Ühendused ja toide"

Commit message: Koomas Plank
Connections:
- net AGND: now also IC2.12 (IO8), IC2.13 (IO19), IC2.14 (IO20), IC2.15 (IO3), IC2.17 (IO9), IC2.18 (IO10), IC2.19 (IO11), IC2.6 (IO6), IC2.7 (IO7), IC2.8 (IO15), IC2.9 (IO16)
Changed lines of the file:
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@@
 	)
 	(junction
+		(at 176.53 119.38)
+		(diameter 0)
+		(color 0 0 0 0)
+	)
+	(junction
+		(at 176.53 99.06)
+		(diameter 0)
+		(color 0 0 0 0)
+	)
+	(junction
+		(at 176.53 114.3)
+		(diameter 0)
+		(color 0 0 0 0)
+	)
+	(junction
 		(at 83.82 165.1)
 		(diameter 0)
@@
 	)
 	(junction
+		(at 176.53 109.22)
+		(diameter 0)
+		(color 0 0 0 0)
+	)
+	(junction
+		(at 176.53 116.84)
+		(diameter 0)
+		(color 0 0 0 0)
+	)
+	(junction
 		(at 107.95 60.96)
 		(diameter 0)
@@
 	)
 	(junction
+		(at 176.53 106.68)
+		(diameter 0)
+		(color 0 0 0 0)
+	)
+	(junction
+		(at 176.53 101.6)
+		(diameter 0)
+		(color 0 0 0 0)
+	)
+	(junction
+		(at 176.53 111.76)
+		(diameter 0)
+		(color 0 0 0 0)
+	)
+	(junction
 		(at 57.15 165.1)
 		(diameter 0)
@@
 	)
 	(junction
+		(at 176.53 96.52)
+		(diameter 0)
+		(color 0 0 0 0)
+	)
+	(junction
 		(at 101.6 53.34)
 		(diameter 0)
@@
 		(color 0 0 0 0)
 	)
+	(junction
+		(at 176.53 104.14)
+		(diameter 0)
+		(color 0 0 0 0)
+	)
 	(wire
 		(pts
@@
 	(wire
 		(pts
+			(xy 176.53 106.68) (xy 176.53 109.22)
+		)
+		(stroke
+			(width 0)
+			(type default)
+		)
+	)
+	(wire
+		(pts
 			(xy 97.79 173.99) (xy 104.14 173.99)
 		)
@@
 	(wire
 		(pts
+			(xy 176.53 99.06) (xy 176.53 101.6)
+		)
+		(stroke
+			(width 0)
+			(type default)
+		)
+	)
+	(wire
+		(pts
 			(xy 109.22 165.1) (xy 109.22 168.91)
 		)
@@
 	(wire
 		(pts
+			(xy 176.53 109.22) (xy 176.53 111.76)
+		)
+		(stroke
+			(width 0)
+			(type default)
+		)
+	)
+	(wire
+		(pts
+			(xy 176.53 96.52) (xy 176.53 99.06)
+		)
+		(stroke
+			(width 0)
+			(type default)
+		)
+	)
+	(wire
+		(pts
 			(xy 140.97 173.99) (xy 144.78 173.99)
 		)
@@
 	(wire
 		(pts
+			(xy 176.53 116.84) (xy 176.53 119.38)
+		)
+		(stroke
+			(width 0)
+			(type default)
+		)
+	)
+	(wire
+		(pts
+			(xy 176.53 119.38) (xy 180.34 119.38)
+		)
+		(stroke
+			(width 0)
+			(type default)
+		)
+	)
+	(wire
+		(pts
 			(xy 101.6 60.96) (xy 107.95 60.96)
 		)
@@
 	(wire
 		(pts
+			(xy 176.53 101.6) (xy 176.53 104.14)
+		)
+		(stroke
+			(width 0)
+			(type default)
+		)
+	)
+	(wire
+		(pts
 			(xy 49.53 67.31) (xy 62.23 67.31)
 		)
@@
 	(wire
 		(pts
+			(xy 176.53 111.76) (xy 176.53 114.3)
+		)
+		(stroke
+			(width 0)
+			(type default)
+		)
+	)
+	(wire
+		(pts
 			(xy 223.52 109.22) (xy 215.9 109.22)
 		)
@@
 	(wire
 		(pts
+			(xy 176.53 93.98) (xy 176.53 96.52)
+		)
+		(stroke
+			(width 0)
+			(type default)
+		)
+	)
+	(wire
+		(pts
 			(xy 132.08 90.17) (xy 143.51 90.17)
 		)
@@
 	(wire
 		(pts
+			(xy 176.53 104.14) (xy 176.53 106.68)
+		)
+		(stroke
+			(width 0)
+			(type default)
+		)
+	)
+	(wire
+		(pts
 			(xy 255.27 119.38) (xy 247.65 119.38)
 		)
@@
 	(wire
 		(pts
+			(xy 176.53 114.3) (xy 176.53 116.84)
+		)
+		(stroke
+			(width 0)
+			(type default)
+		)
+	)
+	(wire
+		(pts
 			(xy 223.52 121.92) (xy 215.9 121.92)
 		)
@@
 	)
 	(symbol
+		(lib_id "power:GND")
+		(at 180.34 119.38 0)
+		(unit 1)
+		(exclude_from_sim no)
+		(in_bom yes)
+		(on_board yes)
+		(dnp no)
+		(fields_autoplaced yes)
+		(property "Reference" "#PWR022"
+			(at 180.34 125.73 0)
+			(effects
+				(font
+					(size 1.27 1.27)
+				)
+				(hide yes)
+			)
+		)
+		(property "Value" "AGND"
+			(at 180.34 124.46 0)
+			(effects
+				(font
+					(size 1.27 1.27)
+				)
+			)
+		)
+		(property "Footprint" ""
+			(at 180.34 119.38 0)
+			(effects
+				(font
+					(size 1.27 1.27)
+				)
+				(hide yes)
+			)
+		)
+		(property "Datasheet" ""
+			(at 180.34 119.38 0)
+			(effects
+				(font
+					(size 1.27 1.27)
+				)
+				(hide yes)
+			)
+		)
+		(property "Description" "Power symbol creates a global label with name \"GND\" , ground"
+			(at 180.34 119.38 0)
+			(effects
+				(font
+					(size 1.27 1.27)
+				)
+				(hide yes)
+			)
+		)
+		(pin "1"
+		)
+		(instances
+			(project "Emaplaat"
+				(path "/489224c0-ace1-4530-aa61-a5d03adf1434"
+					(reference "#PWR022")
+					(unit 1)
+				)
+			)
+		)
+	)
+	(symbol
 		(lib_id "power:VCC")
 		(at 152.4 153.67 0)
@@
 	)
 	(sheet
-		(at 27.305 61.595)
-		(size 22.225 38.1)
+		(at 32.385 61.595)
+		(size 17.145 38.1)
 		(exclude_from_sim no)
 		(in_bom yes)
@@
 		)
 		(property "Sheetname" "uhendused_ja_toide"
-			(at 27.305 60.8834 0)
+			(at 32.385 60.8834 0)
 			(effects
 				(font
@@
 		)
 		(property "Sheetfile" "uhendused_ja_toide.kicad_sch"
-			(at 27.305 100.2796 0)
+			(at 32.385 100.2796 0)
 			(effects
 				(font

Commit message: qwerghhgfdsdfghqwerghhgfdsdfghjj
Parts:
- removed J2, J7: Screw_Terminal_01x02, symbol Connector:Screw_Terminal_01x02
- removed J3, J4: Conn_01x09_Pin, symbol Connector:Conn_01x09_Pin
- C4: renamed from C13; value 0.1u -> 100n
- C5: renamed from C14; value 0.1u -> 100n
- renumbered C10 to C1, C11 to C2, C12 to C3, IC2 to IC1, R2 to R1, R5 to R2, R1 to R3
Connections:
- net !MR1: no longer IC1.22 (IO14)
- net !OE1: no longer IC1.25 (IO48)
- net DS1: no longer IC1.39 (IO1)
- net SHCP1: no longer IC1.23 (IO21)
- net STCP1: no longer IC1.24 (IO47)
- net RX_PULT_1: no longer names the net of IC1.11 (IO18)
- net RX_PULT_2: no longer names the net of IC1.4 (IO4)
- net TX_PULT_1: no longer names the net of IC1.10 (IO17)
- net TX_PULT_2: no longer names the net of IC1.5 (IO5)
- new net !MR2: IC1.22 (IO14)
- new net !OE2: IC1.25 (IO48)
- new net DS2: IC1.39 (IO1)
- new net SHCP2: IC1.23 (IO21)
- new net STCP2: IC1.24 (IO47)
Other:
- added sheet ekraan (ekraan.kicad_sch)
- added sheet ekraan1 (ekraan.kicad_sch)
- sheet uhendused_ja_toide ports: added none; removed RX_pult_1, RX_pult_2, TX_pult_1, TX_pult_2
- note added: "7x14 flipdottide ekraan jagatud kahte ossa"
- note added: "Toite ühendus + üksus ja proge ühendus + üksus"
- note removed: "Sisend ühendused ja toide"
- note removed: "kaks 12V ja GND toite kruvi ühendust 7x7 ekraanidele"
- note removed: "kaks kontroll ühendust 7x7 ekraanidele"
- moved on the sheet: C1, C2, C3, C4, C5, D1, IC1, LS1, Q1, R1, R2, R3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

Commit message: fliptendo gameboy type shi
Parts:
- removed C4, C5: 100n, symbol Device:C
- removed D1: D, symbol Device:D
- removed LS1: KCG0603, KCG0603, symbol KCG0603:KCG0603
- removed Q1: 2N7002K, SOT95P240X120-3N, symbol 2N7002K:2N7002K
- removed R2: 100k, symbol Device:R
- removed R3: 10k, symbol Device:R
- removed S1, S2: TL3305BF100QG, TL3305BF160QG, symbol TL3305BF100QG:TL3305BF100QG
- added D6, D7, D8: LED, LED_SMD:LED_0603_1608Metric, symbol Device:LED
- added NT1: NetTie_2, NetTie:NetTie-2_SMD_Pad0.5mm, symbol Device:NetTie_2
- added R215, R219: 65, Resistor_SMD:R_0603_1608Metric, symbol Device:R
- added R218: 333, Resistor_SMD:R_0603_1608Metric, symbol Device:R
Connections:
- net !MR2: now also IC1.20 (IO12); no longer IC1.22 (IO14)
- net !OE2: now also IC1.23 (IO21); no longer IC1.25 (IO48)
- net 12V: now also D7.2 (A)
- net 3V3: now also D6.2 (A)
- net AGND: now also NT1.2, R215.1, R219.1; no longer IC1.17 (IO9), IC1.18 (IO10), IC1.19 (IO11), IC1.6 (IO6)
- net DS2: now also IC1.24 (IO47); no longer IC1.39 (IO1)
- net PGND: now also NT1.1, R218.1
- net SHCP2: now also IC1.21 (IO13); no longer IC1.23 (IO21)
- net STCP2: now also IC1.22 (IO14); no longer IC1.24 (IO47)
- net flipdot1-: now also IC1.25 (IO48); no longer IC1.38 (IO2)
- net flipdot2+: now also IC1.19 (IO11); no longer IC1.21 (IO13)
- net flipdot2-: now also IC1.18 (IO10); no longer IC1.20 (IO12)
- net Key2: now reaches IC1.10 (IO17)
- net Key1: now reaches IC1.11 (IO18)
- net Key3: now reaches IC1.4 (IO4)
- net Key4: now reaches IC1.5 (IO5)
- new net: D8.1 (K), R219.2
- new net: D6.1 (K), R215.2
- new net: D7.1 (K), R218.2
- new net SW: IC1.6 (IO6)
- new net USER_LED: D8.2 (A), IC1.17 (IO9)
- new net VRX: IC1.39 (IO1)
- new net VRY: IC1.38 (IO2)
Other:
- added sheet perifeeria (perifeeria.kicad_sch)
- note added: "Kõik perifeeria seadmed peale ekraani"
- note added: "indikaator ledid ja PGND - AGND sild"
- note removed: "BOOT ja EN nupud"
- note removed: "Buzzer"
- moved on the sheet: C1, C2, C3, IC1, R1

Commit message: ketamine addict
Parts:
- removed R218: 333, Resistor_SMD:R_0603_1608Metric, symbol Device:R
- added R205: 360, Resistor_SMD:R_0603_1608Metric, symbol Device:R
- R215, R219: value 65 -> 50
Connections:
- net AGND: no longer IC1.12 (IO8), IC1.13 (IO19), IC1.14 (IO20), IC1.15 (IO3), IC1.7 (IO7), IC1.8 (IO15), IC1.9 (IO16)
- net PGND: now also R205.1
- net at D7.1 (K): now also R205.2
- no-connect marks 0 -> 7
Other:
- sheet ekraan ports: added none; removed 12V, 3V3, AGND, PGND
- sheet ekraan1 ports: added none; removed 12V, 3V3, AGND, PGND
- sheet perifeeria ports: added none; removed 3V3, AGND
- sheet uhendused_ja_toide ports: added none; removed 12V, 3V3, AGND, PGND
- note added: "takistid vaja asendada standard mõõdust takistitega"
- moved on the sheet: C1, C2, C3, D7, IC1, NT1, R1

Commit message: T________T Heiki Tammemägi
Parts:
- removed NT1: NetTie_2, NetTie:NetTie-2_SMD_Pad0.5mm, symbol Device:NetTie_2
Connections:
- net PGND is gone; now on net GND: R205.1
- net AGND renamed GND
Other:
- note removed: "takistid vaja asendada standard mõõdust takistitega"
- moved on the sheet: D7, D8, R205, R219
