File: Emaplaat/Emaplaat.kicad_sch (KiCad schematic)
At the start: 15 parts, among them IC1 ESP32-S3-WROOM-2-N32R16V, IC2 74HC595PW-Q100,118, IC3 74HC595PW-Q100,118

Commit message: skeem korras
Parts:
- IC1: footprint ESP32S3WROOM2N32R16V -> ESP32S3WROOM2N32R16V:ESP32S3WROOM2N32R16V
- IC2, IC3: footprint SOP65P640X110-16N -> SOP65P640X110-16N:SOP65P640X110-16N
Changed lines of the file:
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@@
 			)
 		)
-		(property "Footprint" "SOP65P640X110-16N"
+		(property "Footprint" "SOP65P640X110-16N:SOP65P640X110-16N"
 			(at 144.78 223.19 0)
 			(effects
@@
 			)
 		)
-		(property "Footprint" "SOP65P640X110-16N"
+		(property "Footprint" "SOP65P640X110-16N:SOP65P640X110-16N"
 			(at 144.78 258.75 0)
 			(effects
@@
 			)
 		)
-		(property "Footprint" "ESP32S3WROOM2N32R16V"
+		(property "Footprint" "ESP32S3WROOM2N32R16V:ESP32S3WROOM2N32R16V"
 			(at 180.34 140.64 0)
 			(effects

Commit message: :TTT: WWKWKWWKWWKWWKWKWWKWW !"]¤3!E_#1%FV{'14¤#(%2
Connections:
- net BUZZER: now also IC1.9 (IO16)
- no-connect marks 6 -> 5
Changed lines of the file:
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@@
 		(at 184.15 101.6)
 	)
-	(no_connect
-		(at 184.15 96.52)
-	)
 	(wire
 		(pts
@@
 		(pts
 			(xy 151.13 90.17) (xy 140.97 90.17)
+		)
+		(stroke
+			(width 0)
+			(type default)
+		)
+	)
+	(wire
+		(pts
+			(xy 184.15 96.52) (xy 198.12 96.52)
 		)
 		(stroke
@@
 		(effects
 			(font
+				(size 1.27 1.27)
+			)
+			(justify right bottom)
+		)
+	)
+	(label "BUZZER"
+		(at 198.12 96.52 180)
+		(effects
+			(font

Commit message: nig
Connections:
- net !OE: now also IC1.10 (IO17); no longer IC1.17 (IO9)
- net BUZZER: now also IC1.34 (IO41); no longer IC1.9 (IO16)
- net COLUMN1: now also IC1.33 (IO40); no longer IC1.26 (IO45)
- net COLUMN10: now also IC1.21 (IO13); no longer IC1.23 (IO21)
- net COLUMN11: now also IC1.20 (IO12); no longer IC1.22 (IO14)
- net COLUMN12: now also IC1.19 (IO11); no longer IC1.21 (IO13)
- net COLUMN13: now also IC1.18 (IO10); no longer IC1.20 (IO12)
- net COLUMN14: now also IC1.17 (IO9); no longer IC1.19 (IO11)
- net COLUMN2: now also IC1.32 (IO39); no longer IC1.27 (IO0)
- net COLUMN4: now also IC1.27 (IO0); no longer IC1.32 (IO39)
- net COLUMN5: now also IC1.26 (IO45); no longer IC1.33 (IO40)
- net COLUMN6: now also IC1.25 (IO48); no longer IC1.34 (IO41)
- net COLUMN7: now also IC1.24 (IO47); no longer IC1.35 (IO42)
- net COLUMN8: now also IC1.23 (IO21); no longer IC1.25 (IO48)
- net COLUMN9: now also IC1.22 (IO14); no longer IC1.24 (IO47)
- net DS: now also IC1.9 (IO16); no longer IC1.18 (IO10)
- net Key1: now also IC1.5 (IO5); no longer IC1.11 (IO18)
- net Key2: now also IC1.6 (IO6); no longer IC1.10 (IO17)
- net Key4: now also IC1.14 (IO20); no longer IC1.5 (IO5)
- net ROW5_H: now also IC3.2 (Q2); no longer IC3.15 (Q0)
- net ROW6_H: now also IC3.4 (Q4); no longer IC3.2 (Q2)
- net ROW7_H: now also IC3.15 (Q0); no longer IC3.4 (Q4)
- net SHCP: now also IC1.12 (IO8); no longer IC1.14 (IO20)
- net STCP: now also IC1.11 (IO18); no longer IC1.15 (IO3)
- net SW: now also IC1.35 (IO42); no longer IC1.6 (IO6)
- net USER_LED: now also IC1.15 (IO3); no longer IC1.12 (IO8)
- net VRX: now also IC1.38 (IO2); no longer IC1.39 (IO1)
- net VRY: now also IC1.39 (IO1); no longer IC1.38 (IO2)

Commit message: trükkplaat v0 valmis
Connections:
- net ROW1_H: now also IC2.5 (Q5); no longer IC2.15 (Q0)
- net ROW1_L: now also IC2.4 (Q4); no longer IC2.1 (Q1)
- net ROW2_H: now also IC2.7 (Q7); no longer IC2.2 (Q2)
- net ROW2_L: now also IC2.6 (Q6); no longer IC2.3 (Q3)
- net ROW3_H: now also IC2.2 (Q2); no longer IC2.4 (Q4)
- net ROW3_L: now also IC2.3 (Q3); no longer IC2.5 (Q5)
- net ROW4_H: now also IC2.15 (Q0); no longer IC2.6 (Q6)
- net ROW4_L: now also IC2.1 (Q1); no longer IC2.7 (Q7)
Changed lines of the file:
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@@
 	)
 	(label "ROW4_H"
-		(at 157.48 143.51 180)
+		(at 157.48 128.27 180)
 		(effects
 			(font
@@
 	)
 	(label "ROW4_L"
-		(at 157.48 146.05 180)
+		(at 157.48 130.81 180)
 		(effects
 			(font
@@
 	)
 	(label "ROW2_L"
-		(at 157.48 135.89 180)
+		(at 157.48 143.51 180)
 		(effects
 			(font
@@
 	)
 	(label "ROW3_H"
-		(at 157.48 138.43 180)
+		(at 157.48 133.35 180)
 		(effects
 			(font
@@
 	)
 	(label "ROW3_L"
-		(at 157.48 140.97 180)
+		(at 157.48 135.89 180)
 		(effects
 			(font
@@
 	)
 	(label "ROW1_L"
-		(at 157.48 130.81 180)
+		(at 157.48 138.43 180)
 		(effects
 			(font
@@
 	)
 	(label "ROW1_H"
-		(at 157.48 128.27 180)
+		(at 157.48 140.97 180)
 		(effects
 			(font
@@
 	)
 	(label "ROW2_H"
-		(at 157.48 133.35 180)
-		(effects
-			(font
+		(at 157.48 146.05 180)
+		(effects
+			(font

Commit message: trükkplaat v0.1 parandused + 3d failid vaja leid
Parts:
- R4: value 3k -> 3.3k
Changed lines of the file:
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@@
 			)
 		)
-		(property "Value" "3k"
+		(property "Value" "3.3k"
 			(at 70.866 159.004 0)
 			(effects
