File: Emaplaat/ekraan.kicad_sch (KiCad schematic)
At the start: 18 parts, among them IC10 74HC595PW-Q100,118, IC11 74HC595PW-Q100,118, IC13 74HC595PW-Q100,118, IC14 74HC595PW-Q100,118, IC17 74HC595PW-Q100,118, IC20 74HC595PW-Q100,118

Commit message: uuem versioon
Parts:
- removed C31, C33, C37, C39, C49, C55: 47u, symbol Device:C
- removed C32, C34, C38, C40, C50, C56: 100u, symbol Device:C
- removed IC10, IC11, IC13, IC14, IC17, IC20: 74HC595PW-Q100,118, SOP65P640X110-16N, symbol 74HC595PW-Q100_118:74HC595PW-Q100,118
- added C10, C11: 100u, Capacitor_SMD:C_0201_0603Metric_Pad0.64x0.40mm_HandSolder, symbol Device:C
- added D18, D19: D, symbol Device:D
- added IC4, IC5: 1EDN7550BXTSA1, SOT95P280X145-6N, symbol 1EDN7550BXTSA1:1EDN7550BXTSA1
- added R10, R5, R8, R9: 33k, Resistor_SMD:R_0603_1608Metric_Pad0.98x0.95mm_HandSolder, symbol Device:R
Connections:
- net GND: now also C10.1, C11.1, IC4.2 (GND), IC5.2 (GND), R10.2, R8.2
- new net: IC5.1 (IN-), R10.1
- new net: D18.2 (A), IC4.6 (OUT_SNK)
- new net: IC4.3 (IN+), R5.1
- new net: IC5.3 (IN+), R9.1
- new net: D19.1 (K), IC5.5 (OUT_SRC)
- new net: IC4.1 (IN-), R8.1
- new net 12V: C10.2, C11.2, IC4.4 (VDD), IC5.4 (VDD)
- new net E: R5.2, R9.2
Other:
- removed sheet array1
- removed sheet array2
- removed sheet array3
- removed sheet array4
- removed sheet array5
- removed sheet array6
- note removed: "6 nihkeregistrit kontrollimaks 48 flipdot-i"
- note removed: "7x7 flipdot-i"
- note removed: "ühendused + üks pin 49.da flipdoti jaoks"

Commit message: T__T
Parts:
- removed C10, C11: 100u, Capacitor_SMD:C_0201_0603Metric_Pad0.64x0.40mm_HandSolder, symbol Device:C
- removed D18, D19: D, symbol Device:D
- removed IC4, IC5: 1EDN7550BXTSA1, SOT95P280X145-6N, symbol 1EDN7550BXTSA1:1EDN7550BXTSA1
- removed R10, R5, R8, R9: 33k, Resistor_SMD:R_0603_1608Metric_Pad0.98x0.95mm_HandSolder, symbol Device:R
Other:
- removed sheet array
- added sheet Flixlite_maatriks (flixlite_maatriks.kicad_sch)
- added sheet column_signal_to_power (column_signal_to_power.kicad_sch)
- added sheet row_signal_to_power (row_signal_to_power.kicad_sch)
- added sheet row_signal_to_power1 (row_signal_to_power.kicad_sch)
- added sheet row_signal_to_power2 (row_signal_to_power.kicad_sch)
- added sheet row_signal_to_power3 (row_signal_to_power.kicad_sch)
- added sheet row_signal_to_power4 (row_signal_to_power.kicad_sch)
- added sheet row_signal_to_power5 (row_signal_to_power.kicad_sch)
- added sheet row_signal_to_power6 (row_signal_to_power.kicad_sch)
- note added: "Ridade signaalid läbi draiveri"
- note added: "Veergude ja ridade ekraan maatriks"
- note added: "Veergude signaalid läbi draiveri"
