File: Emaplaat/perifeeria.kicad_sch (KiCad schematic)
At the start: 28 parts, among them J3 Conn_01x05_Socket, Q1 2N7002K

Commit message: ts fire commit
Parts:
- removed D10, D11, D12, D13, D14, D5: PESD1ETH10L-QYL, PESD1ETH10LQYL, symbol PESD1ETH10L-QYL:PESD1ETH10L-QYL
- added D10, D11, D12, D13, D14, D5: CPDH3V3UP-HF, SODFL1608X77N, symbol CPDH3V3UP-HF:CPDH3V3UP-HF
Connections:
- net AGND: now also D10. (A), D11. (A), D12. (A), D13. (A), D14. (A), D5. (A)
- net BOOT: now also D13. (A)
- net EN: now also D14. (A)
- net Key1: now also D5. (A)
- net Key2: now also D10. (A)
- net Key3: now also D11. (A)
- net Key4: now also D12. (A)
