File: Emaplaat/Emaplaat.kicad_pcb (KiCad board)
At the start: 2 copper layers, 616 parts, among them IC1 ESP32-S3-WROOM-2-N32R16V, IC10 1EDN7550BXTSA1, IC11 74HC1G04GV-Q100H, IC12 1EDN7550BXTSA1, IC13 74LVC1G66GW,125, IC14 1EDN7550BXTSA1, IC15 74HC1G04GV-Q100H, IC16 1EDN7550BXTSA1, IC17 74LVC1G66GW,125, IC18 1EDN7550BXTSA1, IC19 1EDN7550BXTSA1, IC2 74HC595PW-Q100,118, IC20 1EDN7550BXTSA1, IC21 1EDN7550BXTSA1, IC22 1EDN7550BXTSA1, IC23 1EDN7550BXTSA1, IC24 1EDN7550BXTSA1, IC25 1EDN7550BXTSA1, IC26 1EDN7550BXTSA1, IC27 1EDN7550BXTSA1, IC28 1EDN7550BXTSA1, IC29 1EDN7550BXTSA1, IC3 74HC595PW-Q100,118, IC30 1EDN7550BXTSA1, IC31 1EDN7550BXTSA1, IC32 1EDN7550BXTSA1, IC33 74HC1G04GV-Q100H, IC34 1EDN7550BXTSA1, IC35 74LVC1G66GW,125, IC36 1EDN7550BXTSA1, IC37 74HC1G04GV-Q100H, IC38 1EDN7550BXTSA1, IC39 74LVC1G66GW,125, IC4 TPS54429PWPR, IC40 1EDN7550BXTSA1, IC41 74HC1G04GV-Q100H, IC42 1EDN7550BXTSA1, IC43 74LVC1G66GW,125, IC44 1EDN7550BXTSA1, IC45 74HC1G04GV-Q100H, IC46 1EDN7550BXTSA1, IC47 74LVC1G66GW,125, IC5 FT232RNL-TUBE, IC6 1EDN7550BXTSA1, IC7 74HC1G04GV-Q100H, IC8 1EDN7550BXTSA1, IC9 74LVC1G66GW,125, J1 694108301002, J2 USB4216-03-A, J3 Conn_01x05_Socket, Q1 2N7002K, U1 1EDN7550BXTSA1, U10 1EDN7550BXTSA1, U11 1EDN7550BXTSA1, U12 1EDN7550BXTSA1, U13 1EDN7550BXTSA1, U14 1EDN7550BXTSA1, U2 1EDN7550BXTSA1, U3 1EDN7550BXTSA1, U4 1EDN7550BXTSA1, U5 1EDN7550BXTSA1, U6 1EDN7550BXTSA1, U7 1EDN7550BXTSA1, U8 1EDN7550BXTSA1, U9 1EDN7550BXTSA1

Commit message: trükkplaat valmis võib Abelisle helistada
Other:
- copper layers 2 -> 4
Changed lines of the file:
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@@
 	(generator_version "9.0")
 	(general
-		(thickness 1.6)
+		(thickness 1.600198)
 		(legacy_teardrops no)
 	)
 	(paper "A4")
 	(layers
-		(0 "F.Cu" signal)
-		(2 "B.Cu" signal)
-		(9 "F.Adhes" user "F.Adhesive")
-		(11 "B.Adhes" user "B.Adhesive")
+		(0 "F.Cu" signal "Front")
+		(4 "In1.Cu" signal)
+		(6 "In2.Cu" signal)
+		(2 "B.Cu" signal "Back")
 		(13 "F.Paste" user)
 		(15 "B.Paste" user)
-		(5 "F.SilkS" user "F.Silkscreen")
-		(7 "B.SilkS" user "B.Silkscreen")
+		(5 "F.SilkS" user)
+		(7 "B.SilkS" user)
 		(1 "F.Mask" user)
 		(3 "B.Mask" user)
-		(17 "Dwgs.User" user "User.Drawings")
-		(19 "Cmts.User" user "User.Comments")
-		(21 "Eco1.User" user "User.Eco1")
-		(23 "Eco2.User" user "User.Eco2")
 		(25 "Edge.Cuts" user)
 		(27 "Margin" user)
-		(31 "F.CrtYd" user "F.Courtyard")
-		(29 "B.CrtYd" user "B.Courtyard")
+		(31 "F.CrtYd" user)
+		(29 "B.CrtYd" user)
 		(35 "F.Fab" user)
-		(33 "B.Fab" user)
-		(39 "User.1" user)
-		(41 "User.2" user)
-		(43 "User.3" user)
-		(45 "User.4" user)
 	)
 	(setup
+		(stackup
+			(layer "F.SilkS"
+				(type "Top Silk Screen")
+			)
+			(layer "F.Paste"
+				(type "Top Solder Paste")
+			)
+			(layer "F.Mask"
+				(type "Top Solder Mask")
+				(thickness 0.01)
+			)
+			(layer "F.Cu"
+				(type "copper")
+				(thickness 0.035)
+			)
+			(layer "dielectric 1"
+				(type "core")
+				(thickness 0.480066)
+				(material "FR4")
+				(epsilon_r 4.5)
+				(loss_tangent 0.02)
+			)
+			(layer "In1.Cu"
+				(type "copper")
+				(thickness 0.035)
+			)
+			(layer "dielectric 2"
+				(type "prepreg")
+				(thickness 0.480066)
+				(material "FR4")
+				(epsilon_r 4.5)
+				(loss_tangent 0.02)
+			)
+			(layer "In2.Cu"
+				(type "copper")
+				(thickness 0.035)
+			)
+			(layer "dielectric 3"
+				(type "core")
+				(thickness 0.480066)
+				(material "FR4")
+				(epsilon_r 4.5)
+				(loss_tangent 0.02)
+			)
+			(layer "B.Cu"
+				(type "copper")
+				(thickness 0.035)
+			)
+			(layer "B.Mask"
+				(type "Bottom Solder Mask")
+				(thickness 0.01)
+			)
+			(layer "B.Paste"
+				(type "Bottom Solder Paste")
+			)
+			(layer "B.SilkS"
+				(type "Bottom Silk Screen")
+			)
+			(copper_finish "None")
+			(dielectric_constraints no)
+		)
 		(pad_to_mask_clearance 0)
+		(solder_mask_min_width 0.12)
 		(allow_soldermask_bridges_in_footprints no)
 		(tenting front back)

Commit message: 3 flixli arrayd tehtud
Parts:
- D17, D18, D19, D20, D21, D22, D23, D24, D27, D28, D31, D32, D35, D36, D45, D46, D47, D48, D49, D50, D51, D52, D55, D56, D59, D60, D63, D64, D73, D74, D75, D76, D77, D78, D79, D80, D83, D84, D87, D88, D91, D92: moved to B.Cu
- moved D160 467.7 mm to (549.0, 46.9)
- moved D158 467.5 mm to (549.0, 56.7)
- moved D165 465.6 mm to (548.0, 52.0)
- moved D169 465.6 mm to (548.0, 57.0)
- moved D173 465.6 mm to (548.0, 42.2)
- moved D177 465.6 mm to (548.0, 47.1)
- moved U6 465.6 mm to (544.4, 56.4)
- moved D157 463.7 mm to (546.8, 53.3)
- moved D159 463.5 mm to (546.8, 43.3)
- moved D36 398.4 mm to (340.0, -10.2)
- moved D35 396.9 mm to (337.8, -13.6), turned to 180 degrees
- moved D40 385.7 mm to (338.8, -14.2), turned to 90 degrees
- moved D32 379.8 mm to (339.8, 0.40)
- moved D31 378.6 mm to (338.0, -3.20), turned to 180 degrees
- moved D23 374.2 mm to (337.8, 16.6), turned to 180 degrees
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Routing:
- net /ekraan/COLUMN1_POWER: track 0.00 -> 95.5 mm
- net /ekraan/COLUMN6_POWER: track 74.8 -> 7.57 mm
- net /ekraan/COLUMN2_POWER: track 0.00 -> 26.3 mm
- net /ekraan/COLUMN3_POWER: track 0.00 -> 25.4 mm
- net /ekraan/ROW1_H_POWER: track 5.51 -> 17.7 mm, vias 1 -> 0
- net /ekraan/ROW1_L_POWER: track 6.08 -> 17.7 mm, vias 1 -> 0
- net /ekraan/Flixlite_maatriks/array1/F1: track 0.00 -> 8.93 mm
- net /ekraan/Flixlite_maatriks/array1/G1: track 0.00 -> 8.90 mm
- net /ekraan/Flixlite_maatriks/array1/D1: track 0.00 -> 8.84 mm
- net /ekraan/Flixlite_maatriks/array1/E1: track 0.00 -> 8.84 mm
- net /ekraan/Flixlite_maatriks/array/D1: track 0.00 -> 8.82 mm
- net /ekraan/Flixlite_maatriks/array1/A1: track 0.00 -> 8.79 mm
- net /ekraan/Flixlite_maatriks/array1/C1: track 0.00 -> 8.78 mm
- net /ekraan/Flixlite_maatriks/array1/B1: track 0.00 -> 8.76 mm
- net Net-(D91-K): track 0.00 -> 8.69 mm
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
Commit message: 6 flixel arrayd tehtud
Parts:
- D101, D102, D103, D104, D105, D106, D107, D108, D111, D112, D115, D116, D119, D120, D129, D130, D131, D132, D133, D134, D135, D136, D139, D140, D143, D144, D147, D148, D161, D162, D163, D164, D167, D168, D171, D172, D175, D176: moved to B.Cu
- moved D381 913.0 mm to (1124.5, -1.25)
- moved D382 913.0 mm to (1124.5, 3.10)
- moved D383 913.0 mm to (1124.5, 7.45)
- moved D384 913.0 mm to (1124.5, 11.8)
- moved D385 913.0 mm to (1124.5, 16.1)
- moved D386 913.0 mm to (1124.5, 20.5)
- moved D387 913.0 mm to (1124.5, 24.9)
- moved D389 913.0 mm to (1139.0, -1.80)
- moved D390 913.0 mm to (1139.0, 1.45)
- moved D393 913.0 mm to (1139.0, 4.70)
- moved D394 913.0 mm to (1139.0, 7.95)
- moved D397 913.0 mm to (1139.0, 11.2)
- moved D388 913.0 mm to (1132.2, -1.25)
- moved D391 913.0 mm to (1132.2, 3.10)
- moved D392 913.0 mm to (1132.2, 7.45)
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Routing:
- net /ekraan/COLUMN1_POWER: track 95.5 -> 26.8 mm
- net /ekraan/COLUMN5_POWER: track 0.00 -> 26.2 mm
- net /ekraan/COLUMN4_POWER: track 0.00 -> 26.2 mm
- net /ekraan/COLUMN6_POWER: track 7.57 -> 26.1 mm
- net /ekraan/ROW1_H_POWER: track 17.7 -> 0.00 mm
- net /ekraan/ROW1_L_POWER: track 17.7 -> 0.00 mm
- net /ekraan/Flixlite_maatriks/array3/A1: track 0.00 -> 8.89 mm
- net /ekraan/Flixlite_maatriks/array4/A1: track 0.00 -> 8.89 mm
- net /ekraan/Flixlite_maatriks/array3/B1: track 0.00 -> 8.87 mm
- net /ekraan/Flixlite_maatriks/array4/B1: track 0.00 -> 8.87 mm
- net /ekraan/Flixlite_maatriks/array4/G1: track 0.00 -> 8.85 mm
- net /ekraan/Flixlite_maatriks/array3/G1: track 0.00 -> 8.85 mm
- net /ekraan/Flixlite_maatriks/array3/C1: track 0.00 -> 8.79 mm
- net /ekraan/Flixlite_maatriks/array4/C1: track 0.00 -> 8.79 mm
- net /ekraan/Flixlite_maatriks/array3/F1: track 0.00 -> 8.79 mm
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
Commit message: ekraan maatriks rajad veetud
Parts:
- D185, D186, D187, D188, D189, D190, D191, D192, D195, D196, D199, D200, D203, D204, D213, D214, D215, D216, D217, D218, D219, D220, D223, D224, D227, D228, D231, D232, D241, D242, D243, D244, D245, D246, D247, D248, D251, D252, D255, D256, D259, D260, D269, D270, D271, D272, D273, D274, D275, D276, D279, D280, D283, D284, D287, D288, D297, D298, D299, D300, D301, D302, D303, D304, D307, D308, D311, D312, D315, D316, D325, D326, D327, D328, D329, D330, D331, D332, D335, D336, D339, D340, D343, D344, D353, D354, D355, D356, D357, D358, D359, D360, D363, D364, D367, D368, D371, D372, D381, D382, D383, D384, D385, D386, D387, D388, D391, D392, D395, D396, D399, D400: moved to B.Cu
- moved U14 586.5 mm to (574.4, 63.2)
- moved D405 573.8 mm to (578.3, 43.7), turned to 90 degrees
- moved D408 572.6 mm to (578.3, 33.7), turned to 90 degrees
- moved D407 572.5 mm to (578.3, 29.0), turned to 90 degrees
- moved D406 572.0 mm to (578.3, 2.97), turned to 90 degrees
- moved D401 568.8 mm to (578.3, 54.0), turned to 90 degrees
- moved D403 567.2 mm to (578.3, 38.9), turned to 90 degrees
- moved D404 566.5 mm to (578.3, -1.83), turned to 90 degrees
- moved D398 566.4 mm to (578.3, 8.49), turned to 90 degrees
- moved D402 566.4 mm to (578.3, 13.3), turned to 90 degrees
- moved D389 564.1 mm to (578.3, 59.5), turned to 90 degrees
- moved D393 563.9 mm to (578.3, 64.2), turned to 90 degrees
- moved D397 562.0 mm to (578.3, 49.2), turned to 90 degrees
- moved D390 561.0 mm to (578.3, 18.7), turned to 90 degrees
- moved D394 560.9 mm to (578.3, 23.5), turned to 90 degrees
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Routing:
- net /ekraan/COLUMN7_POWER: track 0.00 -> 26.0 mm
- net /ekraan/COLUMN10_POWER: track 0.00 -> 26.0 mm
- net /ekraan/COLUMN11_POWER: track 0.00 -> 26.0 mm
- net /ekraan/COLUMN9_POWER: track 0.00 -> 26.0 mm
- net /ekraan/COLUMN14_POWER: track 0.00 -> 26.0 mm
- net /ekraan/COLUMN8_POWER: track 0.00 -> 26.0 mm
- net /ekraan/COLUMN12_POWER: track 0.00 -> 26.0 mm
- net /ekraan/COLUMN13_POWER: track 0.00 -> 26.0 mm
- net /ekraan/Flixlite_maatriks/array9/G1: track 0.00 -> 9.36 mm
- net /ekraan/Flixlite_maatriks/array6/G1: track 0.00 -> 9.36 mm
- net /ekraan/Flixlite_maatriks/array12/G1: track 0.00 -> 9.36 mm
- net /ekraan/Flixlite_maatriks/array8/G1: track 0.00 -> 9.36 mm
- net /ekraan/Flixlite_maatriks/array7/G1: track 0.00 -> 9.36 mm
- net /ekraan/Flixlite_maatriks/array13/G1: track 0.00 -> 9.36 mm
- net /ekraan/Flixlite_maatriks/array10/G1: track 0.00 -> 9.36 mm
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