File: Emaplaat/Emaplaat.kicad_pcb (KiCad board)
At the start: 4 copper layers, 616 parts, among them IC1 ESP32-S3-WROOM-2-N32R16V, IC10 1EDN7550BXTSA1, IC11 74HC1G04GV-Q100H, IC12 1EDN7550BXTSA1, IC13 74LVC1G66GW,125, IC14 1EDN7550BXTSA1, IC15 74HC1G04GV-Q100H, IC16 1EDN7550BXTSA1, IC17 74LVC1G66GW,125, IC18 1EDN7550BXTSA1, IC19 1EDN7550BXTSA1, IC2 74HC595PW-Q100,118, IC20 1EDN7550BXTSA1, IC21 1EDN7550BXTSA1, IC22 1EDN7550BXTSA1, IC23 1EDN7550BXTSA1, IC24 1EDN7550BXTSA1, IC25 1EDN7550BXTSA1, IC26 1EDN7550BXTSA1, IC27 1EDN7550BXTSA1, IC28 1EDN7550BXTSA1, IC29 1EDN7550BXTSA1, IC3 74HC595PW-Q100,118, IC30 1EDN7550BXTSA1, IC31 1EDN7550BXTSA1, IC32 1EDN7550BXTSA1, IC33 74HC1G04GV-Q100H, IC34 1EDN7550BXTSA1, IC35 74LVC1G66GW,125, IC36 1EDN7550BXTSA1, IC37 74HC1G04GV-Q100H, IC38 1EDN7550BXTSA1, IC39 74LVC1G66GW,125, IC4 TPS54429PWPR, IC40 1EDN7550BXTSA1, IC41 74HC1G04GV-Q100H, IC42 1EDN7550BXTSA1, IC43 74LVC1G66GW,125, IC44 1EDN7550BXTSA1, IC45 74HC1G04GV-Q100H, IC46 1EDN7550BXTSA1, IC47 74LVC1G66GW,125, IC5 FT232RNL-TUBE, IC6 1EDN7550BXTSA1, IC7 74HC1G04GV-Q100H, IC8 1EDN7550BXTSA1, IC9 74LVC1G66GW,125, J1 694108301002, J2 USB4216-03-A, J3 Conn_01x05_Socket, Q1 2N7002K, U1 1EDN7550BXTSA1, U10 1EDN7550BXTSA1, U11 1EDN7550BXTSA1, U12 1EDN7550BXTSA1, U13 1EDN7550BXTSA1, U14 1EDN7550BXTSA1, U2 1EDN7550BXTSA1, U3 1EDN7550BXTSA1, U4 1EDN7550BXTSA1, U5 1EDN7550BXTSA1, U6 1EDN7550BXTSA1, U7 1EDN7550BXTSA1, U8 1EDN7550BXTSA1, U9 1EDN7550BXTSA1

Commit message: veergude toide veetud
Parts:
- moved R30 519.1 mm to (573.6, -0.12), turned to 180 degrees
- moved R27 511.5 mm to (571.0, -0.28), turned to 90 degrees
- moved R39 506.4 mm to (552.5, -0.28), turned to 90 degrees
- moved R36 505.7 mm to (564.4, -0.12), turned to 180 degrees
- moved C33 503.3 mm to (552.5, 3.24), turned to -90 degrees
- moved C30 501.6 mm to (561.7, 3.24), turned to -90 degrees
- moved R48 501.0 mm to (545.7, -0.12), turned to 180 degrees
- moved C27 500.2 mm to (571.0, 3.24), turned to -90 degrees
- moved R33 498.0 mm to (561.7, -0.28), turned to 90 degrees
- moved IC21 497.8 mm to (564.3, 2.96), turned to -90 degrees
- moved R45 493.2 mm to (543.0, -0.28), turned to 90 degrees
- moved R42 492.4 mm to (555.2, -0.12), turned to 180 degrees
- moved IC18 490.9 mm to (573.5, 2.96), turned to -90 degrees
- moved R28 490.7 mm to (524.5, -0.03), turned to 90 degrees
- moved IC27 490.5 mm to (545.6, 2.96), turned to -90 degrees
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
Commit message: ekraani ridade võim veetud
Parts:
- moved IC13 433.3 mm to (53.1, 113.7)
- moved IC11 427.3 mm to (57.1, 114.3), turned to 90 degrees
- moved R19 426.7 mm to (56.8, 111.2)
- moved IC39 426.4 mm to (53.1, 134.2)
- moved R20 425.7 mm to (61.1, 111.3), turned to 180 degrees
- moved R21 425.4 mm to (64.6, 111.3)
- moved IC37 420.3 mm to (57.1, 135.1), turned to 90 degrees
- moved R62 419.2 mm to (57.0, 132.0)
- moved R63 418.3 mm to (60.8, 132.1), turned to 180 degrees
- moved IC12 417.8 mm to (68.5, 112.3)
- moved R64 417.6 mm to (64.4, 132.1)
- moved R17 416.1 mm to (61.1, 116.6), turned to 180 degrees
- moved R18 415.7 mm to (64.5, 116.6)
- moved IC10 410.6 mm to (68.5, 117.5)
- moved IC38 410.4 mm to (68.4, 133.1)
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
Commit message: algeline paigutus
Parts:
- moved C13 114.9 mm to (60.2, 59.3), turned to 0 degrees
- moved C12 114.7 mm to (60.1, 56.2), turned to 0 degrees
- moved D4 81.7 mm to (97.7, 54.8)
- moved C14 81.7 mm to (88.8, 69.5)
- moved C15 81.7 mm to (88.8, 67.0)
- moved C16 81.7 mm to (88.8, 64.5)
- moved R5 81.7 mm to (88.8, 51.9)
- moved R6 81.7 mm to (84.4, 69.5)
- moved R7 81.7 mm to (84.4, 67.0)
- moved C10 81.7 mm to (93.1, 59.5)
- moved C11 81.7 mm to (93.1, 57.0)
- moved C6 81.7 mm to (93.1, 69.5)
- moved C7 81.7 mm to (93.1, 67.0)
- moved C8 81.7 mm to (93.1, 64.5)
- moved C9 81.7 mm to (93.1, 62.0)
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
Commit message: veel algelisem paigutus
Parts:
- moved R78 59.4 mm to (225.3, 90.0), turned to -90 degrees
- moved R77 58.7 mm to (227.8, 90.0), turned to -90 degrees
- moved R76 55.8 mm to (220.2, 85.7), turned to -90 degrees
- moved R75 54.6 mm to (222.8, 85.7), turned to -90 degrees
- moved C52 50.2 mm to (220.2, 81.3), turned to -90 degrees
- moved R79 49.3 mm to (237.1, 61.8)
- moved C51 48.8 mm to (222.8, 81.3), turned to -90 degrees
- moved C50 47.6 mm to (225.3, 81.3), turned to -90 degrees
- moved C49 46.6 mm to (227.8, 81.3), turned to -90 degrees
- moved D10 45.9 mm to (242.5, 81.0), turned to -90 degrees
- moved D11 45.3 mm to (240.1, 81.0), turned to -90 degrees
- moved D12 44.9 mm to (237.6, 81.0), turned to -90 degrees
- moved D13 44.8 mm to (235.2, 81.0), turned to -90 degrees
- moved D7 43.4 mm to (130.3, 50.8)
- moved D8 43.4 mm to (130.3, 48.3)
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