File: Emaplaat/Emaplaat.kicad_pcb (KiCad board)
At the start: 4 copper layers, 616 parts, among them IC1 ESP32-S3-WROOM-2-N32R16V, IC10 1EDN7550BXTSA1, IC11 74HC1G04GV-Q100H, IC12 1EDN7550BXTSA1, IC13 74LVC1G66GW,125, IC14 1EDN7550BXTSA1, IC15 74HC1G04GV-Q100H, IC16 1EDN7550BXTSA1, IC17 74LVC1G66GW,125, IC18 1EDN7550BXTSA1, IC19 1EDN7550BXTSA1, IC2 74HC595PW-Q100,118, IC20 1EDN7550BXTSA1, IC21 1EDN7550BXTSA1, IC22 1EDN7550BXTSA1, IC23 1EDN7550BXTSA1, IC24 1EDN7550BXTSA1, IC25 1EDN7550BXTSA1, IC26 1EDN7550BXTSA1, IC27 1EDN7550BXTSA1, IC28 1EDN7550BXTSA1, IC29 1EDN7550BXTSA1, IC3 74HC595PW-Q100,118, IC30 1EDN7550BXTSA1, IC31 1EDN7550BXTSA1, IC32 1EDN7550BXTSA1, IC33 74HC1G04GV-Q100H, IC34 1EDN7550BXTSA1, IC35 74LVC1G66GW,125, IC36 1EDN7550BXTSA1, IC37 74HC1G04GV-Q100H, IC38 1EDN7550BXTSA1, IC39 74LVC1G66GW,125, IC4 TPS54429PWPR, IC40 1EDN7550BXTSA1, IC41 74HC1G04GV-Q100H, IC42 1EDN7550BXTSA1, IC43 74LVC1G66GW,125, IC44 1EDN7550BXTSA1, IC45 74HC1G04GV-Q100H, IC46 1EDN7550BXTSA1, IC47 74LVC1G66GW,125, IC5 FT232RNL-TUBE, IC6 1EDN7550BXTSA1, IC7 74HC1G04GV-Q100H, IC8 1EDN7550BXTSA1, IC9 74LVC1G66GW,125, J1 694108301002, J2 USB4216-03-A, J3 Conn_01x05_Socket, Q1 2N7002K, U1 1EDN7550BXTSA1, U10 1EDN7550BXTSA1, U11 1EDN7550BXTSA1, U12 1EDN7550BXTSA1, U13 1EDN7550BXTSA1, U14 1EDN7550BXTSA1, U2 1EDN7550BXTSA1, U3 1EDN7550BXTSA1, U4 1EDN7550BXTSA1, U5 1EDN7550BXTSA1, U6 1EDN7550BXTSA1, U7 1EDN7550BXTSA1, U8 1EDN7550BXTSA1, U9 1EDN7550BXTSA1

Commit message: bonkers
Parts:
- added D10: CPDH3V3UP-HF, Diode_SMD:D_SOD-523, F.Cu at (221.5, 61.1)
- added D11: CPDH3V3UP-HF, Diode_SMD:D_SOD-523, F.Cu at (221.5, 63.6)
- added D12: CPDH3V3UP-HF, Diode_SMD:D_SOD-523, F.Cu at (221.5, 66.0)
- added D13: CPDH3V3UP-HF, Diode_SMD:D_SOD-523, F.Cu at (221.5, 68.5)
- added D4: CPDH3V3UP-HF, Diode_SMD:D_SOD-523, F.Cu at (227.1, 61.1)
- D5, D6: footprint LED_SMD:LED_0603_1608Metric -> LED_SMD:LED_0603_1608Metric_Pad1.05x0.95mm_HandSolder
- moved S6 62.6 mm to (140.0, 56.3), turned to 0 degrees
- moved C53 61.8 mm to (140.0, 50.9)
- moved S5 61.6 mm to (140.0, 46.5), turned to 0 degrees
- moved IC3 61.5 mm to (99.4, 69.5), turned to 0 degrees
- moved C54 59.8 mm to (140.1, 60.7)
- moved D15 59.7 mm to (149.3, 48.7), turned to 90 degrees
- moved D16 57.6 mm to (147.8, 59.1), turned to 90 degrees
- moved IC2 47.9 mm to (112.3, 69.2), turned to 0 degrees
- moved R80 47.8 mm to (147.8, 62.6), turned to 90 degrees
- moved C4 38.9 mm to (136.1, 37.3)
- moved C5 38.9 mm to (136.1, 34.8)
- moved D2 38.9 mm to (131.7, 28.7)
- moved D3 38.9 mm to (131.7, 26.1)
- moved R3 38.9 mm to (136.1, 27.3)
- moved R4 38.9 mm to (136.1, 24.8)
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Connections:
- D15 pad 1: (no net) -> /EN
- D15 pad 2: (no net) -> GND
- D16 pad 1: (no net) -> /BOOT
- D16 pad 2: (no net) -> GND
- D7 pad 1: (no net) -> Net-(D7-K)
- D7 pad 2: (no net) -> GND
- D8 pad 1: (no net) -> Net-(D8-K)
- D8 pad 2: (no net) -> GND
- D9 pad 1: (no net) -> Net-(D9-K)
- D9 pad 2: (no net) -> GND
Routing:
- net /EN: track 0.00 -> 26.1 mm
- net Net-(D7-K): track 0.00 -> 18.1 mm
- net Net-(D8-K): track 0.00 -> 13.0 mm, vias 0 -> 2
- net Net-(J2-CC2): track 0.00 -> 12.7 mm
- net Net-(D9-K): track 0.00 -> 12.2 mm, vias 0 -> 2
- net 3V3: track 0.00 -> 11.1 mm
- net Net-(J2-CC1): track 0.00 -> 10.5 mm
- net Net-(IC5-CBUS1): track 0.00 -> 10.5 mm
- net Net-(IC5-CBUS0): track 0.00 -> 8.23 mm
- net GND: track 0.00 -> 7.03 mm
- net Net-(IC5-3V3OUT): track 0.00 -> 5.38 mm
- net Net-(D6-K): track 0.00 -> 4.22 mm
- net Net-(D5-K): track 0.00 -> 4.22 mm
- net /USER_LED: track 0.00 -> 4.03 mm
- net Net-(D1-K): track 0.00 -> 2.32 mm

Commit message: :TTT: WWKWKWWKWWKWWKWKWWKWW !"]¤3!E_#1%FV{'14¤#(%2
Parts:
- removed the D10 at (242.5, 81.0)
- removed the D11 at (240.1, 81.0)
- removed the D11 at (221.5, 63.6)
- removed the D12 at (237.6, 81.0)
- removed the D13 at (235.2, 81.0)
- removed the D4 at (68.4, 67.7)
- added D11: CPDH3V3UP-HF, Diode_SMD:D_SOD-523, F.Cu at (346.2, 138.8)
- moved IC47 226.5 mm to (234.6, 21.4), turned to 180 degrees
- moved IC45 221.3 mm to (230.7, 20.6), turned to -90 degrees
- moved R70 218.6 mm to (226.9, 18.1), turned to 0 degrees
- moved R72 217.8 mm to (230.9, 23.7), turned to 180 degrees
- moved IC43 214.8 mm to (234.9, 32.2), turned to 180 degrees
- moved R71 213.3 mm to (223.4, 18.1), turned to 180 degrees
- moved C47 211.9 mm to (219.1, 14.6), turned to 180 degrees
- moved R73 211.6 mm to (226.9, 23.6), turned to 0 degrees
- moved J1 209.4 mm to (227.7, 143.4), turned to 90 degrees
- moved IC44 208.9 mm to (219.5, 17.1), turned to 180 degrees
- moved IC41 208.8 mm to (231.0, 31.6), turned to -90 degrees
- moved R74 206.2 mm to (223.4, 23.6), turned to 180 degrees
- moved R67 205.9 mm to (231.3, 34.7), turned to 180 degrees
- moved R65 205.0 mm to (226.9, 29.1), turned to 0 degrees
- moved C48 204.7 mm to (219.2, 19.9), turned to 180 degrees
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Connections:
- IC1 pad 9: unconnected-(IC1-IO16-Pad9) -> /BUZZER
- R75 pad 1: 3V3 -> /Key2
- R75 pad 2: /Key2 -> GND
- R76 pad 1: 3V3 -> /Key1
- R76 pad 2: /Key1 -> GND
- R77 pad 1: 3V3 -> /Key4
- R77 pad 2: /Key4 -> GND
- R78 pad 1: 3V3 -> /Key3
- R78 pad 2: /Key3 -> GND
- S1 pad 1: (no net) -> /Key2
- S1 pad 2: (no net) -> GND
- S2 pad 1: (no net) -> /Key1
- S2 pad 2: (no net) -> GND
- S3 pad 1: (no net) -> /Key4
- S3 pad 2: (no net) -> GND
- S4 pad 1: (no net) -> /Key3
- S4 pad 2: (no net) -> GND
Routing:
- net /EN: track 26.1 -> 0.00 mm
- net Net-(D7-K): track 18.1 -> 0.00 mm
- net Net-(D8-K): track 13.0 -> 0.00 mm, vias 2 -> 0
- net Net-(J2-CC2): track 12.7 -> 0.00 mm
- net Net-(D9-K): track 12.2 -> 0.00 mm, vias 2 -> 0
- net /Key4: track 0.00 -> 11.6 mm
- net 3V3: track 11.1 -> 0.00 mm
- net Net-(J2-CC1): track 10.5 -> 0.00 mm
- net Net-(IC5-CBUS1): track 10.5 -> 0.00 mm
- net /Key1: track 0.00 -> 8.27 mm
- net Net-(IC5-CBUS0): track 8.23 -> 0.00 mm
- net /Key2: track 0.00 -> 8.09 mm
- net /Key3: track 0.00 -> 7.98 mm
- net GND: track 7.03 -> 0.00 mm
- net Net-(IC5-3V3OUT): track 5.38 -> 0.00 mm
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
Commit message: 2
Parts:
- moved C49 146.4 mm to (185.4, 147.3)
- moved C50 146.4 mm to (200.2, 152.8)
- moved C52 146.4 mm to (213.9, 147.8)
- moved D11 146.4 mm to (200.3, 151.1)
- moved D13 146.4 mm to (214.4, 146.1)
- moved S2 146.4 mm to (196.2, 148.2)
- moved S4 146.4 mm to (210.7, 143.1)
- moved C51 146.4 mm to (188.9, 128.5)
- moved D10 146.4 mm to (185.8, 145.6)
- moved D12 146.4 mm to (190.7, 128.1)
- moved R77 146.4 mm to (187.2, 128.5)
- moved S3 146.4 mm to (196.3, 133.9)
- moved R75 146.4 mm to (185.5, 149.1)
- moved R76 146.4 mm to (200.2, 154.6)
- moved R78 146.4 mm to (214.0, 149.6)
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Routing:
- net Net-(D7-K): track 0.00 -> 14.8 mm
- net Net-(D8-K): track 0.00 -> 10.9 mm, vias 0 -> 2
- net Net-(D9-K): track 0.00 -> 10.3 mm, vias 0 -> 2
- net Net-(J2-CC1): track 0.00 -> 9.47 mm, vias 0 -> 2
- net Net-(D14-K): track 0.00 -> 7.86 mm
- net Net-(J2-CC2): track 0.00 -> 5.53 mm
- net Net-(D5-K): track 0.00 -> 1.75 mm
- net Net-(D6-K): track 0.00 -> 1.75 mm

Commit message: nig
Parts:
- moved IC2 84.5 mm to (224.0, 139.6), turned to 90 degrees
- moved C4 84.0 mm to (220.3, 137.4), turned to -90 degrees
- moved C5 76.6 mm to (220.4, 126.8), turned to -90 degrees
- moved IC3 76.1 mm to (224.1, 129.1), turned to 90 degrees
- moved C50 23.0 mm to (180.9, 140.3)
- moved D11 23.0 mm to (181.0, 138.6)
- moved R76 23.0 mm to (180.9, 142.1)
- moved J3 21.9 mm to (103.2, 130.0)
- moved C20 15.4 mm to (94.8, 106.3)
- moved D14 15.4 mm to (108.9, 109.3)
- moved R8 15.4 mm to (94.7, 119.3)
- moved C18 15.4 mm to (89.1, 111.0)
- moved C19 15.4 mm to (90.8, 111.0)
- moved D7 15.4 mm to (86.7, 111.2)
- moved D8 15.4 mm to (88.5, 114.7)
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Connections:
- IC1 pad 10: /Key2 -> /!OE
- IC1 pad 11: /Key1 -> /STCP
- IC1 pad 12: /USER_LED -> /SHCP
- IC1 pad 14: /SHCP -> /Key4
- IC1 pad 15: /STCP -> /USER_LED
- IC1 pad 17: /!OE -> /COLUMN14
- IC1 pad 18: /DS -> /COLUMN13
- IC1 pad 19: /COLUMN14 -> /COLUMN12
- IC1 pad 20: /COLUMN13 -> /COLUMN11
- IC1 pad 21: /COLUMN12 -> /COLUMN10
- IC1 pad 22: /COLUMN11 -> /COLUMN9
- IC1 pad 23: /COLUMN10 -> /COLUMN8
- IC1 pad 24: /COLUMN9 -> /COLUMN7
- IC1 pad 25: /COLUMN8 -> /COLUMN6
- IC1 pad 26: /COLUMN1 -> /COLUMN5
- IC1 pad 27: /COLUMN2 -> /COLUMN4
- IC1 pad 28: Net-(IC1-NC_1) -> unconnected-(IC1-NC_1-Pad28)
- IC1 pad 29: Net-(IC1-NC_1) -> unconnected-(IC1-NC_2-Pad29)
- IC1 pad 30: Net-(IC1-NC_1) -> unconnected-(IC1-NC_3-Pad30)
- IC1 pad 32: /COLUMN4 -> /COLUMN2
- IC1 pad 33: /COLUMN5 -> /COLUMN1
- IC1 pad 34: /COLUMN6 -> /BUZZER
- IC1 pad 35: /COLUMN7 -> /SW
- IC1 pad 38: /VRY -> /VRX
- IC1 pad 39: /VRX -> /VRY
- IC1 pad 5: /Key4 -> /Key1
- IC1 pad 6: /SW -> /Key2
- IC1 pad 9: /BUZZER -> /DS
- IC3 pad 15: /ROW5_H -> /ROW7_H
- IC3 pad 2: /ROW6_H -> /ROW5_H
- IC3 pad 4: /ROW7_H -> /ROW6_H
Routing:
- net 3V3: track 0.00 -> 482.5 mm
- net /ROW7_H: track 0.00 -> 140.4 mm
- net /ekraan/ROW1_H_POWER: track 0.00 -> 140.1 mm, vias 0 -> 4
- net /ekraan/ROW3_H_POWER: track 0.00 -> 140.1 mm, vias 0 -> 4
- net /ekraan/ROW5_H_POWER: track 0.00 -> 140.0 mm, vias 0 -> 4
- net /ekraan/ROW2_H_POWER: track 0.00 -> 140.0 mm, vias 0 -> 4
- net /ekraan/ROW4_H_POWER: track 0.00 -> 139.9 mm, vias 0 -> 4
- net /ekraan/ROW6_L_POWER: track 0.00 -> 139.4 mm, vias 0 -> 4
- net /ekraan/ROW7_L_POWER: track 0.00 -> 139.4 mm, vias 0 -> 4
- net /ekraan/ROW6_H_POWER: track 0.00 -> 139.4 mm, vias 0 -> 4
- net /ekraan/ROW5_L_POWER: track 0.00 -> 138.7 mm, vias 0 -> 4
- net /ekraan/ROW7_H_POWER: track 0.00 -> 138.7 mm, vias 0 -> 4
- net /ekraan/ROW1_L_POWER: track 0.00 -> 138.4 mm, vias 0 -> 4
- net /ekraan/ROW2_L_POWER: track 0.00 -> 138.4 mm, vias 0 -> 4
- net /ekraan/ROW3_L_POWER: track 0.00 -> 138.4 mm, vias 0 -> 4
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- added copper zone on F.Cu, net 12V
