File: Emaplaat/uhendused_ja_toide.kicad_sch (KiCad schematic)
At the start: 33 parts, among them IC16 FT232RNL-TUBE, IC9 TPS54429PWPR, J1 Barrel_Jack, J2 USB4216-03-A

Commit message: toomas plank
Other:
- note removed: "C43 - HF Bypass C44 ja C45 - Decoupler C46 ja C47 - shunt ESDle"
Changed lines of the file:
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@@
-		)
-	)
-	(text "C43 - HF Bypass\nC44 ja C45 - Decoupler\nC46 ja C47 - shunt ESDle"
-		(exclude_from_sim no)
-		(at 122.682 100.33 0)
-		(effects
-			(font
-				(size 1.27 1.27)
-			)
 		)
 	)

Commit message: jajald
Parts:
- removed J1: Barrel_Jack, symbol Connector:Barrel_Jack
- added H1: 0031.8242, 00318242, symbol 00318242:0031.8242
- added J1: 694108301002, 694108301002, symbol 694108301002:694108301002
- C10: renamed from C24; footprint (none) -> Capacitor_SMD:C_0603_1608Metric_Pad1.08x0.95mm_HandSolder
- C11: renamed from C27; footprint (none) -> Capacitor_SMD:C_0603_1608Metric_Pad1.08x0.95mm_HandSolder
- C12: renamed from C25; footprint (none) -> Capacitor_SMD:C_0603_1608Metric_Pad1.08x0.95mm_HandSolder
- C13: renamed from C26; footprint (none) -> Capacitor_SMD:C_0603_1608Metric_Pad1.08x0.95mm_HandSolder
- C14: renamed from C28; footprint (none) -> Capacitor_SMD:C_0603_1608Metric_Pad1.08x0.95mm_HandSolder
- C15: renamed from C29; footprint (none) -> Capacitor_SMD:C_0603_1608Metric_Pad1.08x0.95mm_HandSolder
- C16: renamed from C30; footprint (none) -> Capacitor_SMD:C_0603_1608Metric_Pad1.08x0.95mm_HandSolder
- C17: renamed from C270; footprint (none) -> Capacitor_SMD:C_0603_1608Metric_Pad1.08x0.95mm_HandSolder
- C18: renamed from C12; footprint (none) -> Capacitor_SMD:C_0603_1608Metric_Pad1.08x0.95mm_HandSolder
- C19: renamed from C45; footprint (none) -> Capacitor_SMD:C_0603_1608Metric_Pad1.08x0.95mm_HandSolder
- C20: renamed from C48; footprint (none) -> Capacitor_SMD:C_0603_1608Metric_Pad1.08x0.95mm_HandSolder
- C6: renamed from C20; footprint (none) -> Capacitor_SMD:C_0603_1608Metric_Pad1.08x0.95mm_HandSolder
- C7: renamed from C21; footprint (none) -> Capacitor_SMD:C_0603_1608Metric_Pad1.08x0.95mm_HandSolder
- C8: renamed from C22; footprint (none) -> Capacitor_SMD:C_0603_1608Metric_Pad1.08x0.95mm_HandSolder
- C9: renamed from C23; footprint (none) -> Capacitor_SMD:C_0603_1608Metric_Pad1.08x0.95mm_HandSolder
- L1: footprint (none) -> Inductor_SMD:L_0805_2012Metric_Pad1.05x1.20mm_HandSolder
- R10: renamed from R208; footprint (none) -> Resistor_SMD:R_0603_1608Metric_Pad0.98x0.95mm_HandSolder
- R11: renamed from R209; footprint (none) -> Resistor_SMD:R_0603_1608Metric_Pad0.98x0.95mm_HandSolder
- R5: renamed from R23; footprint (none) -> Resistor_SMD:R_0603_1608Metric_Pad0.98x0.95mm_HandSolder
- R6: renamed from R24; footprint (none) -> Resistor_SMD:R_0603_1608Metric_Pad0.98x0.95mm_HandSolder
- R7: renamed from R25; footprint (none) -> Resistor_SMD:R_0603_1608Metric_Pad0.98x0.95mm_HandSolder
- R8: renamed from R210; footprint Resistor_SMD:R_0603_1608Metric -> Resistor_SMD:R_0603_1608Metric_Pad0.98x0.95mm_HandSolder
- R9: renamed from R211; footprint Resistor_SMD:R_0603_1608Metric -> Resistor_SMD:R_0603_1608Metric_Pad0.98x0.95mm_HandSolder
- renumbered D2 to D4, D15 to D5, D16 to D6, D3 to D7, D4 to D8, IC9 to IC4, IC16 to IC5
Connections:
- net 12V: now also H1.2
- net AGND: now also J1.2
- new net: H1.1, J1.1
- no-connect marks 13 -> 14
Other:
- moved on the sheet: C12, C13, D4

Commit message: skeem korras
Parts:
- D4, D7, D8, D9: footprint SODFL1608X77N -> Diode_SMD:D_SOD-523
- H1: footprint 00318242 -> 00318242:00318242
- IC4: footprint SOP65P640X120-15N -> Package_SO:Texas_HTSSOP-14-1EP_4.4x5mm_P0.65mm_EP3.4x5mm_Mask3.155x3.255mm
- IC5: footprint SOP65P780X200-28N -> SOP65P780X200-28N:SOP65P780X200-28N
- J1: footprint 694108301002 -> 694108301002:694108301002
- J2: footprint USB421603A -> USB421603A:USB421603A

Commit message: väike footprint parandus
Parts:
- D5, D6: footprint LED_SMD:LED_0603_1608Metric -> LED_SMD:LED_0201_0603Metric_Pad0.64x0.40mm_HandSolder
Changed lines of the file:
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@@
 			)
 		)
-		(property "Footprint" "LED_SMD:LED_0603_1608Metric"
+		(property "Footprint" "LED_SMD:LED_0201_0603Metric_Pad0.64x0.40mm_HandSolder"
 			(at 205.74 113.03 0)
 			(effects
@@
 			)
 		)
-		(property "Footprint" "LED_SMD:LED_0603_1608Metric"
+		(property "Footprint" "LED_SMD:LED_0201_0603Metric_Pad0.64x0.40mm_HandSolder"
 			(at 195.58 113.03 0)
 			(effects

Commit message: foot print parandus
Parts:
- D5, D6: footprint LED_SMD:LED_0201_0603Metric_Pad0.64x0.40mm_HandSolder -> LED_SMD:LED_0603_1608Metric_Pad1.05x0.95mm_HandSolder
Changed lines of the file:
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@@
 			)
 		)
-		(property "Footprint" "LED_SMD:LED_0201_0603Metric_Pad0.64x0.40mm_HandSolder"
+		(property "Footprint" "LED_SMD:LED_0603_1608Metric_Pad1.05x0.95mm_HandSolder"
 			(at 205.74 113.03 0)
 			(effects
@@
 			)
 		)
-		(property "Footprint" "LED_SMD:LED_0201_0603Metric_Pad0.64x0.40mm_HandSolder"
+		(property "Footprint" "LED_SMD:LED_0603_1608Metric_Pad1.05x0.95mm_HandSolder"
 			(at 195.58 113.03 0)
 			(effects

Commit message: bonkers
Connections:
- net 12V: now also D4.1 (K); no longer D4. (A)
- net AGND: now also D4.2 (A), D7.2 (A), D8.2 (A), D9.2 (A); no longer D4. (A), D7. (A), D8. (A), D9. (A)
- net at C18.1, C19.1, IC5.20 (VCC)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: now also D7.1 (K); no longer D7. (A)
- net at IC5.15 (USBDP), J2.A6 (DP1), J2.B6 (DP2): now also D9.1 (K); no longer D9. (A)
- net at IC5.16 (USBDM), J2.A7 (DN1), J2.B7 (DN2): now also D8.1 (K); no longer D8. (A)
Changed lines of the file:
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@@
 			)
 		)
-		(pin ""
+		(pin "2"
 		)
-		(pin ""
+		(pin "1"
 		)
 		(instances
@@
 	)
 	(symbol
+		(lib_name "CPDH3V3UP-HF_4")
+		(lib_id "CPDH3V3UP-HF:CPDH3V3UP-HF")
+		(at 76.2 39.37 270)
+		(unit 1)
+		(exclude_from_sim no)
+		(in_bom yes)
+		(on_board yes)
+		(dnp no)
+		(property "Reference" "D4"
+			(at 78.232 46.99 90)
+			(effects
+				(font
+					(size 1.27 1.27)
+				)
+				(justify left)
+			)
+		)
+		(property "Value" "CPDH3V3UP-HF"
+			(at 78.232 49.022 90)
+			(effects
+				(font
+					(size 1.27 1.27)
+				)
+				(justify left)
+			)
+		)
+		(property "Footprint" "Diode_SMD:D_SOD-523"
+			(at -17.45 49.53 0)
+			(effects
+				(font
+					(size 1.27 1.27)
+				)
+				(justify left bottom)
+				(hide yes)
+			)
+		)
+		(property "Datasheet" "https://datasheet.datasheetarchive.com/originals/distributors/Datasheets-DGA26/1842371.pdf"
+			(at -117.45 49.53 0)
+			(effects
+				(font
+					(size 1.27 1.27)
+				)
+				(justify left bottom)
+				(hide yes)
+			)
+		)
+		(property "Description" "ESD Suppressors / TVS Diodes 5.5V, 15Kv"
+			(at 89.916 39.116 0)
+			(effects
+				(font
+					(size 1.27 1.27)
+				)
+				(hide yes)
+			)
+		)
+		(property "Height" "0.77"
+			(at -317.45 49.53 0)
+			(effects
+				(font
+					(size 1.27 1.27)
+				)
+				(justify left bottom)
+				(hide yes)
+			)
+		)
+		(property "Mouser Part Number" "750-CPDH3V3UP-HF"
+			(at -417.45 49.53 0)
+			(effects
+				(font
+					(size 1.27 1.27)
+				)
+				(justify left bottom)
+				(hide yes)
+			)
+		)
+		(property "Mouser Price/Stock" "https://www.mouser.co.uk/ProductDetail/Comchip-Technology/CPDH3V3UP-HF?qs=XEIV%2Fho1H6em2DT135enQw%3D%3D"
+			(at -517.45 49.53 0)
+			(effects
+				(font
+					(size 1.27 1.27)
+				)
+				(justify left bottom)
+				(hide yes)
+			)
+		)
+		(property "Manufacturer_Name" "Comchip Technology"
+			(at -617.45 49.53 0)
+			(effects
+				(font
+					(size 1.27 1.27)
+				)
+				(justify left bottom)
+				(hide yes)
+			)
+		)
+		(property "Manufacturer_Part_Number" "CPDH3V3UP-HF"
+			(at -717.45 49.53 0)
+			(effects
+				(font
+					(size 1.27 1.27)
+				)
+				(justify left bottom)
+				(hide yes)
+			)
+		)
+		(pin "1"
+		)
+		(pin "2"
+		)
+		(instances
+			(project "Emaplaat"
+				(path "/489224c0-ace1-4530-aa61-a5d03adf1434/902edf26-f9ad-46ee-8658-d4b7491aa9c7"
+					(reference "D4")
+					(unit 1)
+				)
+			)
+		)
+	)
+	(symbol
 		(lib_id "power:VCC")
 		(at 133.35 38.1 0)
@@
 			)
 		)
-		(pin ""
+		(pin "1"
 		)
-		(pin ""
+		(pin "2"
 		)
 		(instances
@@
 	)
 	(symbol
-		(lib_name "CPDH3V3UP-HF_3")
-		(lib_id "CPDH3V3UP-HF:CPDH3V3UP-HF")
-		(at 76.2 39.37 270)
-		(unit 1)
-		(exclude_from_sim no)
-		(in_bom yes)
-		(on_board yes)
-		(dnp no)
-		(property "Reference" "D4"
-			(at 78.232 46.99 90)
-			(effects
-				(font
-					(size 1.27 1.27)
-				)
-				(justify left)
-			)
-		)
-		(property "Value" "CPDH3V3UP-HF"
-			(at 78.232 49.53 90)
-			(effects
-				(font
-					(size 1.27 1.27)
-				)
-				(justify left)
-			)
-		)
-		(property "Footprint" "Diode_SMD:D_SOD-523"
-			(at -17.45 49.53 0)
-			(effects
-				(font
-					(size 1.27 1.27)
-				)
-				(justify left bottom)
-				(hide yes)
-			)
-		)
-		(property "Datasheet" "https://datasheet.datasheetarchive.com/originals/distributors/Datasheets-DGA26/1842371.pdf"
-			(at -117.45 49.53 0)
-			(effects
-				(font
-					(size 1.27 1.27)
-				)
-				(justify left bottom)
-				(hide yes)
-			)
-		)
-		(property "Description" "ESD Suppressors / TVS Diodes 5.5V, 15Kv"
-			(at 89.916 39.116 0)
-			(effects
-				(font
-					(size 1.27 1.27)
-				)
-				(hide yes)
-			)
-		)
-		(property "Height" "0.77"
-			(at -317.45 49.53 0)
-			(effects
-				(font
-					(size 1.27 1.27)
-				)
-				(justify left bottom)
-				(hide yes)
-			)
-		)
-		(property "Mouser Part Number" "750-CPDH3V3UP-HF"
-			(at -417.45 49.53 0)
-			(effects
-				(font
-					(size 1.27 1.27)
-				)
-				(justify left bottom)
-				(hide yes)
-			)
-		)
-		(property "Mouser Price/Stock" "https://www.mouser.co.uk/ProductDetail/Comchip-Technology/CPDH3V3UP-HF?qs=XEIV%2Fho1H6em2DT135enQw%3D%3D"
-			(at -517.45 49.53 0)
-			(effects
-				(font
-					(size 1.27 1.27)
-				)
-				(justify left bottom)
-				(hide yes)
-			)
-		)
-		(property "Manufacturer_Name" "Comchip Technology"
-			(at -617.45 49.53 0)
-			(effects
-				(font
-					(size 1.27 1.27)
-				)
-				(justify left bottom)
-				(hide yes)
-			)
-		)
-		(property "Manufacturer_Part_Number" "CPDH3V3UP-HF"
-			(at -717.45 49.53 0)
-			(effects
-				(font
-					(size 1.27 1.27)
-				)
-				(justify left bottom)
-				(hide yes)
-			)
-		)
-		(pin ""
-		)
-		(pin ""
-		)
-		(instances
-			(project "Emaplaat"
-				(path "/489224c0-ace1-4530-aa61-a5d03adf1434/902edf26-f9ad-46ee-8658-d4b7491aa9c7"
-					(reference "D4")
-					(unit 1)
-				)
-			)
-		)
-	)
-	(symbol
 		(lib_id "power:GND")
 		(at 153.67 96.52 0)
@@
 			)
 		)
-		(pin ""
+		(pin "2"
 		)
-		(pin ""
+		(pin "1"
 		)
 		(instances

Commit message: trükkplaat v0.1 parandused + 3d failid vaja leid
Parts:
- added R81: 18k, Resistor_SMD:R_0603_1608Metric_Pad0.98x0.95mm_HandSolder, symbol Device:R
- R6: value 73.2k -> 56k
- R7: value 22.1k -> 22k
- R8, R9: value 360 -> 330
Connections:
- net 12V: no longer D4.1 (K)
- net at C14.2, IC4.2 (VFB), R7.1: now also R81.2; no longer R6.2
- net at H1.1, J1.1: now also D4.1 (K)
- new net: R6.2, R81.1
Other:
- moved on the sheet: C12, C13, D4, H1, R7

Commit message: v1.0 aga muudatusi on vaja veel teha
Parts:
- C12: symbol Device:C -> Device:C_Polarized
- C14: value 20p -> 22p
- D4: Voltage (none) -> 3.3V
Changed lines of the file:
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@@
+			)
+		)
+		(property "Voltage" "3.3V"
+			(at 64.262 51.308 90)
+			(effects
+				(font
+					(size 1.27 1.27)
+				)
 			)
 		)
@@
 	)
 	(symbol
-		(lib_id "Device:C")
+		(lib_id "Device:C_Polarized")
 		(at 93.98 48.26 0)
 		(unit 1)
@@
 			)
 		)
-		(property "Description" "Unpolarized capacitor"
+		(property "Description" "Polarized capacitor"
 			(at 93.98 48.26 0)
 			(effects
@@
 			)
 		)
-		(property "Value" "20p"
+		(property "Value" "22p"
 			(at 152.4 59.6899 0)
 			(effects
