File: Emaplaat/array.kicad_sch (KiCad schematic)
At the start: 1 part, among them U2 1EDN7550BXTSA1

Commit message: T__T
Parts:
- added D409, D410, D411, D412, D413, D414, D415, D416, D419, D420, D423, D424, D427, D428: D_Zener, symbol Device:D_Zener
- added D417, D418, D421, D422, D425, D426, D429, D430, D431, D432, D433, D434, D435, D436: D, symbol Device:D
- renumbered U2 to U15
Connections:
- net FLIXEL_A renamed A1
- net A1: now also D409.2 (A), D417.1 (K), D421.2 (A)
- net FLIXEL_B renamed B1
- net B1: now also D411.2 (A), D425.1 (K), D429.2 (A)
- net FLIXEL_C renamed C1
- net C1: now also D413.2 (A), D431.1 (K), D433.2 (A)
- net FLIXEL_D renamed D1
- net D1: now also D415.2 (A), D435.1 (K), D436.2 (A)
- net FLIXEL_E renamed E1
- net E1: now also D418.1 (K), D419.2 (A), D422.2 (A)
- net FLIXEL_F renamed F1
- net F1: now also D423.2 (A), D426.1 (K), D430.2 (A)
- net FLIXEL_G renamed G1
- net G1: now also D427.2 (A), D432.1 (K), D434.2 (A)
- net GND renamed COLUMN_POWER
- net COLUMN_POWER: now also D410.2 (A), D412.2 (A), D414.2 (A), D416.2 (A), D420.2 (A), D424.2 (A), D428.2 (A)
- new net: D423.1 (K), D424.1 (K)
- new net: D415.1 (K), D416.1 (K)
- new net: D413.1 (K), D414.1 (K)
- new net: D409.1 (K), D410.1 (K)
- new net: D411.1 (K), D412.1 (K)
- new net: D427.1 (K), D428.1 (K)
- new net: D419.1 (K), D420.1 (K)
- new net ROW1_HIGH_POWER: D417.2 (A)
- new net ROW1_LOW_POWER: D421.1 (K)
- new net ROW2_HIGH_POWER: D425.2 (A)
- new net ROW2_LOW_POWER: D429.1 (K)
- new net ROW3_HIGH_POWER: D431.2 (A)
- new net ROW3_LOW_POWER: D433.1 (K)
- new net ROW4_HIGH_POWER: D435.2 (A)
- new net ROW4_LOW_POWER: D436.1 (K)
- new net ROW5_HIGH_POWER: D418.2 (A)
- new net ROW5_LOW_POWER: D422.1 (K)
- new net ROW6_HIGH_POWER: D426.2 (A)
- new net ROW6_LOW_POWER: D430.1 (K)
- new net ROW7_HIGH_POWER: D432.2 (A)
- new net ROW7_LOW_POWER: D434.1 (K)
Other:
- note added: "12V Zener dioodid, et induktoreid kaitsta"
- note added: "Diodiid et individuaalselt flixleid kontrollida"
- note added: "Flixlite kogum"
- note added: "Veerul on ühine punkt"
- note removed: "1x7 Flipdot-id kogum"
- moved on the sheet: U15

Commit message: jajald
Parts:
- removed D410, D411, D412, D413, D414, D415, D416, D419, D420, D423, D424, D427, D428: D_Zener, symbol Device:D_Zener
- removed D418, D421, D422, D425, D426, D429, D430, D431, D432, D433, D434, D435, D436: D, symbol Device:D
- added D18, D19, D20, D21, D22, D23, D24, D27, D28, D31, D32, D35, D36: D_Zener, DO-214AC-2: DO-214AC-2, symbol Device:D_Zener
- added D26, D29, D30, D33, D34, D37, D38, D39, D40, D41, D42, D43, D44: D, SOD-123FL:SOD-123FL, symbol Device:D
- D17: renamed from D409; footprint (none) -> DO-214AC-2: DO-214AC-2
- D25: renamed from D417; footprint (none) -> SOD-123FL:SOD-123FL
- renumbered U15 to U1
Connections:
- net A1: now also D29.2 (A)
- net B1: now also D19.2 (A), D33.1 (K), D37.2 (A)
- net C1: now also D21.2 (A), D39.1 (K), D41.2 (A)
- net COLUMN_POWER: now also D18.2 (A), D20.2 (A), D22.2 (A), D24.2 (A), D28.2 (A), D32.2 (A), D36.2 (A)
- net D1: now also D23.2 (A), D43.1 (K), D44.2 (A)
- net E1: now also D26.1 (K), D27.2 (A), D30.2 (A)
- net F1: now also D31.2 (A), D34.1 (K), D38.2 (A)
- net G1: now also D35.2 (A), D40.1 (K), D42.2 (A)
- net ROW1_LOW_POWER: now also D29.1 (K)
- net ROW2_HIGH_POWER: now also D33.2 (A)
- net ROW2_LOW_POWER: now also D37.1 (K)
- net ROW3_HIGH_POWER: now also D39.2 (A)
- net ROW3_LOW_POWER: now also D41.1 (K)
- net ROW4_HIGH_POWER: now also D43.2 (A)
- net ROW4_LOW_POWER: now also D44.1 (K)
- net ROW5_HIGH_POWER: now also D26.2 (A)
- net ROW5_LOW_POWER: now also D30.1 (K)
- net ROW6_HIGH_POWER: now also D34.2 (A)
- net ROW6_LOW_POWER: now also D38.1 (K)
- net ROW7_HIGH_POWER: now also D40.2 (A)
- net ROW7_LOW_POWER: now also D42.1 (K)
- net at D17.1 (K): now also D18.1 (K)
- new net: D19.1 (K), D20.1 (K)
- new net: D31.1 (K), D32.1 (K)
- new net: D27.1 (K), D28.1 (K)
- new net: D23.1 (K), D24.1 (K)
- new net: D35.1 (K), D36.1 (K)
- new net: D21.1 (K), D22.1 (K)

Commit message: v3.3 Abeltoni tagasiside veelkord
Changed lines of the file:
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@@
 		(fields_autoplaced yes)
 		(property "Reference" "U1"
-			(at 165.6293 78.8353 0)
+			(at 165.735 78.74 0)
 			(effects
 				(font
@@
 		)
 		(property "Value" "1EDN7550BXTSA1"
-			(at 165.6293 81.3753 0)
+			(at 165.735 81.28 0)
 			(effects
 				(font
