File: Flipdot_Simulatsioon/Flipdot_Simulatsioon.kicad_sch (KiCad schematic)
At the start: 4 parts

Commit message: jajald
Parts:
- removed C1: 100u, symbol Device:C
Connections:
- net at R1.1: now also V1.1
Other:
- moved on the sheet: L1, R1
Changed lines of the file:
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@@
 	(wire
 		(pts
-			(xy 123.19 181.61) (xy 125.73 181.61)
+			(xy 107.95 181.61) (xy 110.49 181.61)
 		)
 		(stroke
@@
 	(wire
 		(pts
-			(xy 125.73 181.61) (xy 125.73 184.15)
+			(xy 110.49 181.61) (xy 110.49 185.42)
 		)
 		(stroke
@@
 	(wire
 		(pts
-			(xy 82.55 181.61) (xy 92.71 181.61)
+			(xy 82.55 181.61) (xy 88.9 181.61)
 		)
 		(stroke
@@
 	(wire
 		(pts
-			(xy 100.33 181.61) (xy 104.14 181.61)
-		)
-		(stroke
-			(width 0)
-			(type default)
-		)
-	)
-	(wire
-		(pts
-			(xy 111.76 181.61) (xy 115.57 181.61)
+			(xy 96.52 181.61) (xy 100.33 181.61)
 		)
 		(stroke
@@
 	(symbol
 		(lib_id "Simulation_SPICE:0")
-		(at 125.73 184.15 0)
+		(at 110.49 185.42 0)
 		(unit 1)
 		(exclude_from_sim no)
@@
 		(dnp no)
 		(property "Reference" "#GND02"
-			(at 125.73 189.23 0)
+			(at 110.49 190.5 0)
 			(effects
 				(font
@@
 		)
 		(property "Value" "0"
-			(at 129.032 182.372 0)
+			(at 113.792 183.642 0)
 			(effects
 				(font
@@
 		)
 		(property "Footprint" ""
-			(at 125.73 184.15 0)
+			(at 110.49 185.42 0)
 			(effects
 				(font
@@
 		)
 		(property "Datasheet" "https://ngspice.sourceforge.io/docs/ngspice-html-manual/manual.xhtml#subsec_Circuit_elements__device"
-			(at 125.73 194.31 0)
+			(at 110.49 195.58 0)
 			(effects
 				(font
@@
 		)
 		(property "Description" "0V reference potential for simulation"
-			(at 125.73 191.77 0)
+			(at 110.49 193.04 0)
 			(effects
 				(font
@@
 	(symbol
 		(lib_id "Device:R")
-		(at 107.95 181.61 90)
+		(at 92.71 181.61 90)
 		(unit 1)
 		(exclude_from_sim no)
@@
 		(fields_autoplaced yes)
 		(property "Reference" "R1"
-			(at 107.95 175.26 90)
+			(at 92.71 175.26 90)
 			(effects
 				(font
@@
 		)
 		(property "Value" "18"
-			(at 107.95 177.8 90)
+			(at 92.71 177.8 90)
 			(effects
 				(font
@@
 		)
 		(property "Footprint" ""
-			(at 107.95 183.388 90)
+			(at 92.71 183.388 90)
 			(effects
 				(font
@@
 		)
 		(property "Datasheet" "~"
-			(at 107.95 181.61 0)
+			(at 92.71 181.61 0)
 			(effects
 				(font
@@
 		)
 		(property "Description" "Resistor"
-			(at 107.95 181.61 0)
+			(at 92.71 181.61 0)
 			(effects
 				(font
@@
 	)
 	(symbol
-		(lib_id "Device:C")
-		(at 96.52 181.61 90)
-		(unit 1)
-		(exclude_from_sim no)
-		(in_bom yes)
-		(on_board yes)
-		(dnp no)
-		(fields_autoplaced yes)
-		(property "Reference" "C1"
-			(at 96.52 173.99 90)
-			(effects
-				(font
-					(size 1.27 1.27)
-				)
-			)
-		)
-		(property "Value" "100u"
-			(at 96.52 176.53 90)
-			(effects
-				(font
-					(size 1.27 1.27)
-				)
-			)
-		)
-		(property "Footprint" ""
-			(at 100.33 180.6448 0)
-			(effects
-				(font
-					(size 1.27 1.27)
-				)
-				(hide yes)
-			)
-		)
-		(property "Datasheet" "~"
-			(at 96.52 181.61 0)
-			(effects
-				(font
-					(size 1.27 1.27)
-				)
-				(hide yes)
-			)
-		)
-		(property "Description" "Unpolarized capacitor"
-			(at 96.52 181.61 0)
-			(effects
-				(font
-					(size 1.27 1.27)
-				)
-				(hide yes)
-			)
-		)
-		(pin "1"
-		)
-		(pin "2"
-		)
-		(instances
-			(project ""
-				(path "/718663e9-5efc-4ad6-a482-03fb8ef1cf6c"
-					(reference "C1")
-					(unit 1)
-				)
-			)
-		)
-	)
-	(symbol
 		(lib_id "Device:L")
-		(at 119.38 181.61 90)
+		(at 104.14 181.61 90)
 		(unit 1)
 		(exclude_from_sim no)
@@
 		(fields_autoplaced yes)
 		(property "Reference" "L1"
-			(at 119.38 176.53 90)
+			(at 104.14 176.53 90)
 			(effects
 				(font
@@
 		)
 		(property "Value" "6m"
-			(at 119.38 179.07 90)
+			(at 104.14 179.07 90)
 			(effects
 				(font
@@
 		)
 		(property "Footprint" ""
-			(at 119.38 181.61 0)
+			(at 104.14 181.61 0)
 			(effects
 				(font
@@
 		)
 		(property "Datasheet" "~"
-			(at 119.38 181.61 0)
+			(at 104.14 181.61 0)
 			(effects
 				(font
@@
 		)
 		(property "Description" "Inductor"
-			(at 119.38 181.61 0)
+			(at 104.14 181.61 0)
 			(effects
 				(font
@@
 			)
 		)
-		(property "Sim.Params" "y1=0 y2=12 td=2n tr=15n tf=15n tw=33m per=66m"
+		(property "Sim.Params" "y1=0 y2=10.9 td=2n tr=15n tf=15n tw=1m per=4m"
 			(at 86.36 167.7697 0)
 			(effects
